File: rtcl-pmod-hub75e/rtcl-pmod-hub75e.kicad_sch (KiCad schematic)
At the start: 22 parts, among them J1 PMOD, J2 HUB75E, J3 Conn_01x02, U1 74LVC273, U2 74LVC273, U3 74LVC273, U4 74LVC273, U5 LM809M3-2.93, U6 SN74LVC2G86DCUR

Commit message: Add new footprints for SPDT switch and OS102011MS2QN1 switch
- Created a new footprint for SPDT switch (SPDT_OS102011_CNK) with detailed pad and silk layer definitions.
- Added a new footprint for OS102011MS2QN1 switch, including properties, pads, and 3D model reference.
Parts:
- added R3: 10k, Resistor_SMD:R_0603_1608Metric, symbol Device:R
- added SW1: OS102011MS2QN1, rtcl-pmod-hub75e:SW_OS102011MS2QN1, symbol Switch:SW_SPDT
- U5: value LM809M3-2.93 -> APX803D-29SAG-7; footprint Package_TO_SOT_SMD:SOT-23 -> Package_TO_SOT_SMD:SOT-23-3; LCSC C414611 -> C460555
Connections:
- net +3.3V: now also R3.2
- net GND: now also SW1.3 (C)
- net RESET: now also R3.1, SW1.2 (B)
- no-connect marks 0 -> 1

Commit message: Update README and add LCSC part number for OS102011MS2QN1 switch
Parts:
- SW1: LCSC (none) -> C221829
Changed lines of the file:
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@@
+			)
+		)
+		(property "LCSC" "C221829"
+			(at 93.98 99.06 0)
+			(hide yes)
+			(show_name no)
+			(do_not_autoplace no)
+			(effects
+				(font
+					(size 1.27 1.27)
+				)
 			)
 		)
